Commit message: minor changes

File: software/ros2_ws/src/arm_teleop/urdf/dicerox_arm.urdf (robot description, URDF)
Before this commit: robot Dicerox_robot_arm_URDF, 8 links, 7 joints
Links:
- link Link1: geometry collision mesh filename=package://arm_teleop/meshes/collision/Link1.stl; visual mesh filename=package://arm_teleop/meshes/visual/Link1.STL
- link Link2: geometry collision mesh filename=package://arm_teleop/meshes/collision/Link2.stl; visual mesh filename=package://arm_teleop/meshes/visual/Link2.STL
- link Link3: geometry collision mesh filename=package://arm_teleop/meshes/collision/Link3.stl; visual mesh filename=package://arm_teleop/meshes/visual/Link3.STL
- link Link4: geometry collision mesh filename=package://arm_teleop/meshes/collision/Link4.stl; visual mesh filename=package://arm_teleop/meshes/visual/Link4.STL
- link Link5: geometry collision mesh filename=package://arm_teleop/meshes/collision/Link5.stl; visual mesh filename=package://arm_teleop/meshes/visual/Link5.STL
- link Link6: geometry collision mesh filename=package://arm_teleop/meshes/collision/Link6.stl; visual mesh filename=package://arm_teleop/meshes/visual/Link6.STL
